Commit message: for Preliminary Match

File: burger_war/models/burgerbot.gazebo.xacro (robot description, xacro)
@@ -42,8 +42,8 @@
   <gazebo>
     <plugin name="turtlebot3_burger_controller" filename="libgazebo_ros_diff_drive.so">
-      <commandTopic>cmd_vel</commandTopic>
+      <commandTopic>limited_cmd_vel</commandTopic>
       <odometryTopic>odom</odometryTopic>
       <odometryFrame>odom</odometryFrame>
-      <odometrySource>encoder</odometrySource>
+      <odometrySource>world</odometrySource>
       <publishOdomTF>true</publishOdomTF>
       <robotBaseFrame>base_footprint</robotBaseFrame>
@@ -162,5 +162,11 @@
   </gazebo>
   <gazebo reference="poll">
-    <material>Gazebo/DarkGrey</material>
+    <material>Gazebo/White</material>
+  </gazebo>
+  <gazebo reference="blue_plate">
+    <material>Gazebo/Blue</material>
+  </gazebo>
+  <gazebo reference="red_plate">
+    <material>Gazebo/Red</material>
   </gazebo>
 </robot>
